File: kicad/featherwing_qcopter/featherwing_qcopter.kicad_pcb (KiCad board)
At the start: 2 copper layers, 86.4 x 86.4 mm, 42 parts, among them J1 Conn_01x16_Male, J2 Conn_01x12_Male, J3 Motor connector, J4 Motor connector, J5 Motor connector, J6 Motor connector, U1 DRV8837CDSGR, U2 DRV8837CDSGR, U3 DRV8837CDSGR, U4 DRV8837CDSGR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

Commit message: repository updated
Parts:
- moved C14 40.2 mm to (146.3, 119.3)
- moved C15 40.2 mm to (146.3, 117.4)
- moved C16 40.2 mm to (144.5, 115.1)
- moved D1 40.2 mm to (121.3, 116.8)
- moved J3 40.2 mm to (114.3, 88.9)
- moved U3 40.2 mm to (155.1, 131.0)
- moved C1 40.2 mm to (120.5, 101.5)
- moved C10 40.2 mm to (158.9, 129.2)
- moved C12 40.2 mm to (141.6, 110.2)
- moved C13 40.2 mm to (136.5, 110.2)
- moved C7 40.2 mm to (158.9, 133.0)
- moved D2 40.2 mm to (158.1, 116.8)
- moved J1 40.2 mm to (129.5, 95.2)
- moved R1 40.2 mm to (121.5, 108.3)
- moved R10 40.2 mm to (156.2, 116.8)
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Connections:
- C6 pad 1: Net-(C6-Pad1) -> +3V3
- U5 pad 4: Net-(C6-Pad1) -> +3V3
Routing:
- net +3V3: track 223.6 -> 236.2 mm
- net Net-(C6-Pad1): track 6.87 -> 0.00 mm
Other:
- board text added: "featherwing_copter iman_201912.02"
- board text removed: "featherwing_copter iman_201912.01"
